File: Circuits/motherboard/pinchy.sch (EAGLE design)
At the start: 49 parts, among them J1 Tenacita, J10 AN3, J11 AN4, J12 AN5, J15 POWER_JACKPTH, J19 Utrasonic, J2 OptoreflectorA, J20 Analogicas, J21 Bluetooth, J22 Alimentacion, J3 ServoA, J4 ServoB, J5 OptoreflectorB, J6 D13, J7 AN0, J8 AN1, J9 AN2, Q1 BC847, SW1 MFP106D, SW2 EVQQ2, U1 TPS63061DSCT, U2 MAX7219CWG+, U3 LM555D

Commit message: ❌ Deleted unused files
Parts:
- removed J22: Alimentacion, pinhead:PINHD-1X3
- removed J23, J24: (no value), pinhead:PINHD-1X17
- removed J25: (no value), pinhead:PINHD-1X2
- added C10, C12: 1uF/X5R/16V, rcl:C-EUC1206
- added C11, C18, C7, C8, C9: 0.1uF/X5R/6V3, rcl:C-EUC0805
- added C13: 10uF/Tan/25V, lib_Pinchy:C1206-POL
- added C14, C19: 22uF/tan/6V3, lib_Pinchy:C1206-POL
- added C15, C16: 12pF/NP0, rcl:C-EUC0805
- added C17: 0.1uF/X5R/6V3, rcl:C-EUC1206
- added D2: SSB43L, lib_Pinchy:SSB43L
- added D3, D4: PMEG3030EP, diode:SCHOTTKY-DIODESMD
- added D5, D6: BAT54C, diode:BAT54C
- added D7: Yellow TX LED, adafruit:LEDCHIPLED_0805
- added D8: Yellow RX LED, adafruit:LEDCHIPLED_0805
- added D9: GREEN PWR_ON, adafruit:LEDCHIPLED_0805
- added J14: ZX62D-B-5PA8(30), lib_Pinchy:ZX62D-B-5PA8(30)
- added J18: JST RCY, pinhead:PINHD-1X2
- added L2: EMI 742792012, WE-CBF:WE-CBF-742792012_0805
- added L3: MH2029-300Y, rcl:R-EU_R0805
- added Q2: DMP3098L, zetex:PMOSSOT23
- added Q3, Q4: DMP2035U-7, zetex:PMOSSOT23
- added R11, R19: 82k, rcl:R-EU_R0805
- added R12, R20: 18k, rcl:R-EU_R0805
- added R13: 4K7, rcl:R-EU_R0805
- added R15, R16, R18: 1k, rcl:R-EU_R0805
- added R17, R22, R27: 10k, rcl:R-EU_R0805
- added R21: 51k, rcl:R-EU_R0805
- added R25, R26: VARISTORCN0603, varistor:VARISTORCN0603
- added RN1: 22R, resistor-dil:4R-NCAY16
- added SW3: MFP106D, mk2:MFP106D
- added U4: ATMEGA32U4-AU, adafruit:ATMEGA32U4-AU
- added U5: LM1117MPX-5.0, lm1117:LM1117MPX-5.0
- added U6: LM1117MPX-3.3, pinchy:LM1117MPX-3.3
- added U7: LMV358, linear:LM358D
- added WIFI1: ESP8622-12E, lib_Pinchy:ESP8622-12E
- added XTAL: 16MHz, adafruit:XTAL-4-3225
- C1: value 100uF -> 47uF/X5R/6.3V; device Jaegger_MKII:EDK107M016A9G -> rcl:C-EUC1210
- C2: value 100uF -> 10uF/X5R/25V; device Jaegger_MKII:EDK107M016A9G -> rcl:C-EUC0805
- C3, C6: value 0.1uF -> 0.1uF/X5R/6V3
- C4: value 0.1uF -> 10uF/Tan/25V; device rcl:C-EUC0805 -> lib_Pinchy:C1206-POL
- C5: value 220nF -> 220nF/X5R/6V3
- F1: value SMD260F -> MF-MSMF050-2
- J13: value (none) -> I/O
- J16: value (none) -> ICSP; device SparkFun-Connectors:M06SILK_FEMALE_PTH -> pinhead:PINHD-2X3
- J17: value (none) -> Matrix; device SparkFun-Connectors:M06SILK_FEMALE_PTH -> pinhead:PINHD-1X5
- J21: value Bluetooth -> Alimentacion; device pinhead:PINHD-1X4 -> pinhead:PINHD-1X3
- L1: value 1uH -> 4.7uH; device Jaegger_MKII:MCSDRH73B -> lib_Pinchy:TDK_VLF10040T_4R7N5R4
- R1: value 62k -> 100k
- R2: value 10k -> 4K7
- SW1: value MFP106D -> EVQQ2; device mk2:MFP106D -> mk2:JAEGGER_MKII_EVQQ2
- U1: value TPS63061DSCT -> ADP2303ARDZ-5.0; device Jaegger_MKII:TPS63061DSCT -> lib_Pinchy:ADP2303ARDZ-5.0
- U2: value MAX7219CWG+ -> TCA9406DCTR; device maxim7219:MAX7219CWG+ -> lib_Pinchy:TCA9406DCTR
Connections:
- removed net 3.3V: J22.2, J24.16
- removed net C1: J17.1, U2.SEG_A
- removed net C2: J17.3, U2.SEG_B
- removed net C3: J16.3, U2.SEG_C
- removed net C4: J16.6, U2.SEG_D
- removed net C5: J16.5, U2.SEG_E
- removed net D14: J24.2, R7.1, SW2.P$2
- removed net R1: J16.1, U2.DIG_0
- removed net R2: J16.2, U2.DIG_1
- removed net R3: J17.2, U2.DIG_2
- removed net R4: J16.4, U2.DIG_3
- removed net R5: J17.4, U2.DIG_4
- removed net R6: J17.5, U2.DIG_5
- removed net R7: J17.6, U2.DIG_6
- new net +3.3V: C19.+, J21.2, R13.2, U2.OE, U2.VCCA, U6.OUT, U6.OUT1, WIFI1.GPIO2, WIFI1.VCC
- new net +5V_REG: C14.+, C7.1, C8.1, D9.A, J16.2, L3.1, Q3.D, R22.2, U2.VCCB, U4.AVCC1, U4.UVCC, U4.VCC, U4.VCC1, U5.OUT, U5.OUT1
- new net D14/MISO: J16.1, R7.1, SW2.P$2, U4.PB3(PDO/MISO)
- new net HWB: R17.1, U4.PE2(!HWB)
- new net N$16: R2.1, WIFI1.GPIO15
- new net N$18: J14.D+, R25.2, RN1B.2
- new net N$19: J14.D-, R26.2, RN1A.2
- new net N$20: D6.A1, J15.PWR, J18.1, Q2.S
- new net N$21: D5.CC, Q4.G, R21.2
- new net N$25: R11.1, R12.2, U7A.+IN, U7B.+IN
- new net N$27: C3.1, U1.BST
- new net N$29: D5.A1, Q3.G, U7A.OUT
- new net N$30: C15.1, U4.XTAL1, XTAL.X1
- new net N$31: C16.1, U4.XTAL2, XTAL.X2
- new net N$34: C10.1, U4.UCAP
- new net N$35: C12.1, L3.2, U4.AVCC
- new net N$38: D8.A, R15.2
- new net N$40: Q2.G, SW3.COM
- new net N$42: D6.CC, SW3.1
- new net N$44: C13.+, D4.C, U5.IN
- new net N$46: D9.C, R18.2
- new net N$47: D7.A, R16.2
- new net N$48: D5.A2, U7B.OUT
- new net N$49: R19.1, R20.2, U7A.-IN, U7B.-IN
- new net RD_N: RN1A.1, U4.D-
- new net RD_P: RN1B.1, U4.D+
- new net RESET: J16.5, R22.1, SW1.P$2, U4./RESET
- new net RXD_3.3: U2.SCL_A, WIFI1.RXD
- new net TXD_3.3: U2.SDA_A, WIFI1.TXD
- new net TX_LED: R16.1, U4.PD5(XCK/CTS)
- new net U4: C11.1, U4.AREF
- new net VUSB: C17.1, C18.1, C9.1, D6.A2, F1.2, Q3.S, Q4.S, R19.2, R27.2, U4.VBUS, U7P.V+
- net +5V: now also C1.1, C4.+, J17.1, L1.2, Q4.D, U6.IN; no longer C2.1, C4.1, J22.1, J24.6, R1.2, U1.VOUT, U2.V+
- net A0: now also U4.PF7(ADC7(TDI); no longer J24.14
- net A1: now also U4.PF6(ADC6/TDO); no longer J24.13
- net A2: now also U4.PF5(ADC5/TMS); no longer J24.12
- net A3: now also U4.PF4(ADC4/TCK); no longer J24.11
- net A4: now also U4.PF1(ADC1); no longer J24.10
- net A5: now also U4.PF0(ADC0); no longer J24.9
- net D0/RX: now also U2.SDA_B, U4.PD2(INT2/RXD1); no longer J21.3, J23.4
- net D1/TX: now also U2.SCL_B, U4.PD3(INT3/TXD1); no longer J21.4, J23.3
- net D10: now also U4.PB6(OC1B/OC4B/ADC13); no longer J23.15
- net D11: now also U4.PB7(OC0A/OC1C/RTS); no longer J23.16
- net D12: now also U4.PD6(T1/ADC9/!OC4D); no longer J23.17
- net D13: now also U4.PC7(ICP3/CLK0/OC4A); no longer J24.17
- net D15/SCK: now also J16.3, J17.4, U4.PB1(SCK); no longer J24.1, U2.CLK
- net D16/MOSI: now also J16.4, J17.2, U4.PB2(PDI/MOSI); no longer J23.1, U2.DIN
- net D17/SS: now also J17.3, R15.1, U4.PB0(SS); no longer J23.2, R2.2, U2.LOAD
- net D2: now also U4.PD1(INT1/SDA); no longer J23.7
- net D3: now also U4.PD0(INT0/OC0B/SCL); no longer J23.8
- net D4: now also U4.PD4(ICP1/ADC8); no longer J23.9
- net D5: now also U4.PC6(OC3A/!OC4A); no longer J23.10
- net D6: now also U4.PD7(OC4D/ADC10/T0); no longer J23.11
- net D7: now also U4.PE6(INT.6/AIN0); no longer J23.12
- net D8: now also U4.PB4(ADC11); no longer J23.13
- net D9: now also U4.PB5(OC1A/ADC12/!OC4B); no longer J23.14
- net GND: now also C10.2, C11.2, C12.2, C13.-, C14.-, C15.2, C16.2, C17.2, C18.2, C19.-, C4.-, C7.2, C8.2, C9.2, D2.A, D7.C, D8.C, J14.GND, J16.6, J17.5, J18.2, J21.3, R12.1, R17.2, R18.1, R2.2, R20.1, R21.1, R25.1, R26.1, R27.1, SW1.P$1, SW3.2, U4.GND, U4.GND1, U4.GND2, U4.GND3, U4.UGND, U5.GND, U6.GND, U7P.V-, WIFI1.GND, XTAL.G1, XTAL.G2; no longer C3.2, C4.2, J21.2, J22.3, J24.4, J25.2, R2.1, U1.PGND, U1.PS/SYNC, U2.GND_2
- net N$12: now also C3.2, D2.C, L1.1, U1.SW; no longer F1.1, SW1.2
- net N$22: now also F1.1, J14.VUSB; no longer R1.1, U2.ISET
- net N$23: now also L2.1, Q2.D; no longer J15.PWR, J25.1, SW1.COM
- net N$5: now also C2.1, D3.C, R1.2, U1.EN, U1.VIN; no longer C3.1, U1.VAUX
- net N$8: now also R13.1, WIFI1.EN; no longer L1.P$2, U1.L1
- net N$9: now also R1.1, U1.PGOOD; no longer L1.P$1, U1.L2
- net VCC: now also D3.A, D4.A, L2.2, R11.2; no longer C1.1, F1.2, U1.EN, U1.VIN
Other:
- note added: "555 Oscilator 2.8Khz"
- note added: "Buck Fixed 5V para alimentación de potencia Regulador de tensión fixed a 5V para el microncontrolador Regulador de tensión fixed a 3V3 para el modulo WIFI"
- note added: "Buzzer"
- note added: "Entradas de alimentación Switch On-Off Filtro EMI"
- note added: "I/O Female Header"
- note added: "I/O Male Header"
- note added: "ICSP"
- note added: "Led RGB"
- note added: "Matrix Connector"
- note added: "NC"
- note added: "Pull Up Button"
- note added: "Selector de tension -Si está el USB conectado y no la alimentacion externa, los nMos están conduciendo y todo el circuito tiene VUSB -Si está el USB conectado y la alimentacion externa, los pMos están cerrados -Si no está el USB conectado y si la alimentacion externa, los nMos están cerrados"
- note added: "USB Connector"
- note added: "WIFI"
